File: Switch.kicad_sch (KiCad schematic)
At the start: 110 parts, among them J10 C1,2, J11 C1,2, J12 C1,2, J3 C1,2, J4 C1,2, J5 C1,2, J6 C1,2, J7 C1,2, J8 C1,2, J9 C1,2, Q1 NMOS, Q10 NMOS, Q11 NMOS, Q12 NMOS, Q13 NMOS, Q14 NMOS, Q15 NMOS, Q16 NMOS, Q17 NMOS, Q18 NMOS, Q19 NMOS, Q2 NMOS, Q20 NMOS, Q3 NMOS, Q4 NMOS, Q5 NMOS, Q6 NMOS, Q7 NMOS, Q8 NMOS, Q9 NMOS

Commit message: updated Routing
Parts:
- D10, D11, D12, D13, D14, D15, D16, D17, D18, D19, D20, D21, D22, D23, D4, D5, D6, D7, D8, D9: footprint (none) -> LED_SMD:LED_0603_1608Metric
- J10, J11, J12, J3, J4, J5, J6, J7, J8, J9: footprint (none) -> TerminalBlock_Phoenix:TerminalBlock_Phoenix_MKDS-3-2-5.08_1x02_P5.08mm_Horizontal
- Q1, Q10, Q11, Q12, Q13, Q14, Q15, Q16, Q17, Q18, Q19, Q2, Q20, Q3, Q4, Q5, Q6, Q7, Q8, Q9: value NMOS -> MOT90N03D; footprint (none) -> Package_TO_SOT_SMD:TO-252-2; symbol Simulation_SPICE:NMOS -> locallib:MOT90N03D; mpn (none) -> MOT90N03D
- R10, R12, R13, R15, R16, R18, R19, R25, R26, R27, R28, R29, R30, R31, R32, R33, R34, R40, R41, R42, R43, R44, R45, R46, R47, R48, R49, R55, R56, R57, R58, R59, R6, R60, R61, R62, R63, R64, R7, R9: footprint (none) -> Resistor_SMD:R_0603_1608Metric
- R11, R14, R17, R20, R21, R22, R23, R24, R35, R36, R37, R38, R39, R5, R50, R51, R52, R53, R54, R8: value 220R -> 240R; footprint (none) -> Resistor_SMD:R_0603_1608Metric
Connections:
- net PA0 is gone; now on net PA3: R5.1
- net PA1 is gone; now on net PA4: R8.1
- net PA2 is gone; now on net PA5: R11.1
- net CH1: now also J3.1 (Pin_1), Q1.2 (D); no longer J3.2 (Pin_2), Q1.1 (D)
- net CH10: now also J7.2 (Pin_2), Q9.2 (D); no longer J7.1 (Pin_1), Q9.1 (D)
- net CH11: now also Q12.2 (D); no longer Q12.1 (D)
- net CH12: now also Q15.2 (D); no longer Q15.1 (D)
- net CH13: now also Q11.2 (D); no longer Q11.1 (D)
- net CH14: now also Q13.2 (D); no longer Q13.1 (D)
- net CH15: now also Q14.2 (D); no longer Q14.1 (D)
- net CH16: now also Q17.2 (D); no longer Q17.1 (D)
- net CH17: now also Q20.2 (D); no longer Q20.1 (D)
- net CH18: now also Q16.2 (D); no longer Q16.1 (D)
- net CH19: now also Q18.2 (D); no longer Q18.1 (D)
- net CH2: now also J3.2 (Pin_2), Q2.2 (D); no longer J3.1 (Pin_1), Q2.1 (D)
- net CH20: now also Q19.2 (D); no longer Q19.1 (D)
- net CH3: now also J4.1 (Pin_1), Q3.2 (D); no longer J4.2 (Pin_2), Q3.1 (D)
- net CH4: now also J4.2 (Pin_2), Q4.2 (D); no longer J4.1 (Pin_1), Q4.1 (D)
- net CH5: now also J5.1 (Pin_1), Q5.2 (D); no longer J5.2 (Pin_2), Q5.1 (D)
- net CH6: now also J5.2 (Pin_2), Q7.2 (D); no longer J5.1 (Pin_1), Q7.1 (D)
- net CH7: now also J6.1 (Pin_1), Q10.2 (D); no longer J6.2 (Pin_2), Q10.1 (D)
- net CH8: now also J6.2 (Pin_2), Q6.2 (D); no longer J6.1 (Pin_1), Q6.1 (D)
- net CH9: now also J7.1 (Pin_1), Q8.2 (D); no longer J7.2 (Pin_2), Q8.1 (D)
- net PA10: now also R37.1; no longer R36.1
- net PA3: no longer R14.1
- net PA4: no longer R17.1
- net PA5: no longer R21.1
- net PA6: now also R14.1; no longer R24.1
- net PA7: now also R17.1; no longer R20.1
- net PA8: now also R51.1; no longer R22.1
- net PA9: now also R38.1; no longer R23.1
- net PB0: now also R21.1; no longer R39.1
- net PB1: now also R24.1; no longer R35.1
- net PB10: now also R22.1; no longer R38.1
- net PB11: now also R23.1; no longer R51.1
- net PB12: now also R53.1; no longer R54.1
- net PB13: now also R52.1; no longer R50.1
- net PB14: now also R50.1; no longer R52.1
- net PB15: now also R54.1; no longer R53.1
- net PB2: now also R20.1; no longer R37.1
- net at R51.2, R56.2: now also Q17.1 (G); no longer Q17.2 (G)
- net at R8.2, R9.2: now also Q2.1 (G); no longer Q2.2 (G)
- net at R17.2, R18.2: now also Q5.1 (G); no longer Q5.2 (G)
- net at R50.2, R55.2: now also Q16.1 (G); no longer Q16.2 (G)
- net at R54.2, R59.2: now also Q20.1 (G); no longer Q20.2 (G)
- net at R5.2, R6.2: now also Q1.1 (G); no longer Q1.2 (G)
- net at R36.2, R41.2: now also Q12.1 (G); no longer Q12.2 (G)
- net at R39.2, R44.2: now also Q15.1 (G); no longer Q15.2 (G)
- net at R38.2, R43.2: now also Q14.1 (G); no longer Q14.2 (G)
- net at R20.2, R25.2: now also Q6.1 (G); no longer Q6.2 (G)
- net at R14.2, R15.2: now also Q4.1 (G); no longer Q4.2 (G)
- net at R24.2, R29.2: now also Q10.1 (G); no longer Q10.2 (G)
- net at R52.2, R57.2: now also Q18.1 (G); no longer Q18.2 (G)
- net at R22.2, R27.2: now also Q8.1 (G); no longer Q8.2 (G)
- net at R35.2, R40.2: now also Q11.1 (G); no longer Q11.2 (G)
- net at R53.2, R58.2: now also Q19.1 (G); no longer Q19.2 (G)
- net at R37.2, R42.2: now also Q13.1 (G); no longer Q13.2 (G)
- net at R23.2, R28.2: now also Q9.1 (G); no longer Q9.2 (G)
- net at R21.2, R26.2: now also Q7.1 (G); no longer Q7.2 (G)
- net at R11.2, R12.2: now also Q3.1 (G); no longer Q3.2 (G)
- new net PA11: R35.1
- new net PA12: R39.1
- new net PB9: R36.1
Other:
- moved on the sheet: J3, J4, J5, J6, J7
